Commit message: 왼쪽벽 인식

File: mastering_ros_robot_description_pkg/urdf/seven_dof_arm.urdf (robot description, URDF)
Before this commit: robot seven_dof_arm, 12 links, 11 joints
Links:
- link grasping_frame: geometry visual box size=0.01 0.01 0.01

File: mastering_ros_robot_description_pkg/urdf/seven_dof_arm.xacro (robot description, xacro)
@@ -144,5 +144,5 @@
   </link>
   <gazebo reference="shoulder_pan_link">
-    <material>Gazebo/Red</material>
+    <material>Gazebo/Blue</material>
   </gazebo>
   <joint name="shoulder_pitch_joint" type="revolute">
@@ -320,5 +320,5 @@
   </link>
   <gazebo reference="gripper_roll_link">
-    <material>Gazebo/Red</material>
+    <material>Gazebo/Blue</material>
   </gazebo>
   <joint name="finger_joint1" type="prismatic">
